File: eagle/stm32f4_sd.brd (EAGLE design)
At the start: 48 x 24.5 mm, 36 parts, among them IC1 STM32F405RGT, IC2 LT1763CS8-3.3, SW1 SWITCH_MCTAEF, U1 USD-SOCKETNEW

Commit message: minor updates
Parts:
- added LED3: (no value), SparkFun-LED:LED-0603
- added R6: 150R, rcl:R0402
- LED1, LED2: device led:CHIPLED_0805 -> SparkFun-LED:LED-0603
- U1: value USD-SOCKETNEW -> 2908-05WB-MG
- moved LED1 0.97 mm to (41.5, 12.3)
- moved R2 0.97 mm to (44.8, 12.3)
- moved C5 0.92 mm to (2.40, 18.2), turned to 180 degrees
- moved LED2 0.70 mm to (41.5, 10.9)
- moved R3 0.70 mm to (44.8, 10.9)
- moved R1 0.30 mm to (38.4, 6.20)
- moved SW1 0.10 mm to (43.3, 17.7)
Connections:
- new net N$1: IC1.35, LED3.C
- new net N$6: LED3.A, R6.2
- net +3V3: now also R6.1
- net B14: now also IC1.36; no longer IC1.35
- net B15: now also IC1.37; no longer IC1.36
- net BOOT: now also IC1.24
- net C6: now also IC1.38; no longer IC1.37
- net C7: now also IC1.39; no longer IC1.38
- net C8: now also IC1.40; no longer IC1.39
Routing:
- net N$1: track 0.00 -> 6.52 mm
- net BOOT: track 47.2 -> 53.3 mm
- net +5V: track 72.5 -> 67.0 mm
- net +3V3: track 125.3 -> 129.5 mm
- net N$6: track 0.00 -> 1.95 mm
- net N$26: track 5.34 -> 6.71 mm
- net N$15: track 5.78 -> 6.84 mm
- net GND: vias 33 -> 34
Other:
- board size 48 x 24.5 mm -> 48 x 24.6 mm
- board text added: "1"
- board text added: "2"
- board text added: "3"
- board text added: "C9"
- board text removed: "B14"
