File: eagle/stm32f4_sd.sch (EAGLE design)
At the start: 36 parts, among them IC1 STM32F405RGT, IC2 LT1763CS8-3.3, SW1 SWITCH_MCTAEF, U1 USD-SOCKETNEW

Commit message: minor updates
Parts:
- added LED3: (no value), SparkFun-LED:LED0603
- added R6: 150R, rcl:R-EU_R0402
- LED1, LED2: device led:LEDCHIPLED_0805 -> SparkFun-LED:LED0603
- U1: value USD-SOCKETNEW -> 2908-05WB-MG; 3M (none) -> 2908-05WB-MG
Connections:
- new net N$1: IC1.PB14, LED3.C
- new net N$6: LED3.A, R6.2
- net +3V3: now also R6.1
- net B14: now also IC1.PB15; no longer IC1.PB14
- net B15: now also IC1.PC6; no longer IC1.PB15
- net BOOT: now also IC1.PC4
- net C6: now also IC1.PC7; no longer IC1.PC6
- net C7: now also IC1.PC8; no longer IC1.PC7
- net C8: now also IC1.PC9; no longer IC1.PC8
Other:
- note added: "new SD Product: SCHA4B0400"
- moved on the sheet: SW1
